File: 555 timer.kicad_pcb (KiCad board)
At the start: 2 copper layers, 39.7 x 31.3 mm, 11 parts, among them J1 Screw_Terminal_01x02, J2 Conn_01x02_Male, T1 LMC555xM

Commit message: Design modifications
Parts:
- added REF**: MountingHole_2.2mm_M2, MountingHole:MountingHole_2.2mm_M2, F.Cu at (41.4, -612.9)
- J2: footprint Connector_PinHeader_1.00mm:PinHeader_1x02_P1.00mm_Vertical -> Connector_PinSocket_2.00mm:PinSocket_1x02_P2.00mm_Vertical
Routing:
- net GND: track 105.0 -> 20.5 mm, vias 0 -> 8
- net Net-(D3-Pad2): track 90.3 -> 74.0 mm
- net Net-(D3-Pad1): track 14.1 -> 29.9 mm
- net Net-(C2-Pad1): track 9.77 -> 11.4 mm
- net Net-(J1-Pad2): track 33.9 -> 32.5 mm
Other:
- net class Default: trace_width 0.2 -> 0.13
