File: 555 timer.sch (KiCad schematic (older format))
At the start: 11 parts, among them J1 Screw_Terminal_01x02, J2 Conn_01x02_Male, T1 LMC555xM

Commit message: Design modifications
Parts:
- J2: footprint Connector_PinHeader_1.00mm:PinHeader_1x02_P1.00mm_Vertical -> Connector_PinSocket_2.00mm:PinSocket_1x02_P2.00mm_Vertical
Changed lines of the file:
@@
 F 0 "J2" H 8100 3500 50  0000 C CNN
 F 1 "Conn_01x02_Male" H 8050 3250 50  0000 C CNN
-F 2 "Connector_PinHeader_1.00mm:PinHeader_1x02_P1.00mm_Vertical" H 8000 3450 50  0001 C CNN
+F 2 "Connector_PinSocket_2.00mm:PinSocket_1x02_P2.00mm_Vertical" H 8000 3450 50  0001 C CNN
 F 3 "~" H 8000 3450 50  0001 C CNN
 	1    8000 3450
